Commit message: camera traseira

File: robutler_description_23-24/urdf/robutler.gazebo.xacro (robot description, xacro)
@@ -6,4 +6,10 @@
   <gazebo reference="base_link">
     <material>Gazebo/Red</material>
+  </gazebo>
+   <gazebo reference="new_camera_link">
+    <material>Gazebo/Red</material>
+  </gazebo>
+   <gazebo reference="new_camera_base_link">
+    <material>Gazebo/FlatBlack</material>
   </gazebo>
   <gazebo reference="wheel_left_link">
@@ -168,3 +174,37 @@
     </sensor>
   </gazebo>
+  <gazebo reference="camera_rgb_frame2">
+    <sensor type="camera" name="Pi Camera2">
+      <always_on>true</always_on>
+      <pose>0 0 0 0 0 3.14159</pose>
+      <visualize>$(arg camera_visual)</visualize>
+      <camera>
+          <horizontal_fov>1.085595</horizontal_fov>
+          <!-- <horizontal_fov>2.085595</horizontal_fov> -->
+          <image>
+              <width>640</width>
+              <height>480</height>
+              <format>R8G8B8</format>
+          </image>
+          <clip>
+              <near>0.03</near>
+              <far>100</far>
+          </clip>
+      </camera>
+      <plugin name="camera_controller" filename="libgazebo_ros_camera.so">
+        <alwaysOn>true</alwaysOn>
+        <updateRate>30.0</updateRate>
+        <cameraName>camera2</cameraName>
+        <frameName>camera_rgb_optical_frame2</frameName>
+        <imageTopicName>rgb/image_raw2</imageTopicName>
+        <cameraInfoTopicName>rgb/camera_info2</cameraInfoTopicName>
+        <hackBaseline>0.07</hackBaseline>
+        <distortionK1>0.0</distortionK1>
+        <distortionK2>0.0</distortionK2>
+        <distortionK3>0.0</distortionK3>
+        <distortionT1>0.0</distortionT1>
+        <distortionT2>0.0</distortionT2>
+      </plugin>
+    </sensor>
+  </gazebo>
 </robot>

File: robutler_description_23-24/urdf/robutler.urdf.xacro (robot description, xacro)
@@ -213,4 +213,16 @@
     <child link="new_camera_base_link"/>
   </joint>
+  <joint name="new_camera_rgb_joint" type="fixed">
+    <origin xyz="-0.06 0 0.6" rpy="0 0 3.14159"/>
+    <parent link="new_camera_base_link"/>
+    <child link="camera_rgb_frame2"/>
+  </joint>
+  <link name="camera_rgb_frame2"/>
+  <joint name="new_camera_rgb_optical_joint" type="fixed">
+    <origin xyz="0 0 0" rpy="-1.57 0 -1.57"/>
+    <parent link="camera_rgb_frame2"/>
+    <child link="camera_rgb_optical_frame2"/>
+  </joint>
+  <link name="camera_rgb_optical_frame2"/>
   <joint name="camera_rgb_joint" type="fixed">
     <origin xyz="0.003 0.011 0.009" rpy="0 0 0"/>

Commit message: a

File: robutler_description_23-24/urdf/robutler.gazebo.xacro (robot description, xacro)
@@ -177,5 +177,5 @@
     <sensor type="camera" name="Pi Camera2">
       <always_on>true</always_on>
-      <pose>0 0 0 0 0 3.14159</pose>
+      <pose>0 0 0 0 0 0</pose>
       <visualize>$(arg camera_visual)</visualize>
       <camera>

File: robutler_description_23-24/urdf/robutler.urdf.xacro (robot description, xacro)
@@ -214,5 +214,5 @@
   </joint>
   <joint name="new_camera_rgb_joint" type="fixed">
-    <origin xyz="-0.06 0 0.6" rpy="0 0 3.14159"/>
+    <origin xyz="-0.06 0 0.6" rpy="0 0 0"/>
     <parent link="new_camera_base_link"/>
     <child link="camera_rgb_frame2"/>
