Commit message: l

File: robutler_description_23-24/urdf/robutler.urdf.xacro (robot description, xacro)
@@ -174,15 +174,42 @@
   </link>
   <link name="new_camera_link">
-    <collision>
-      <origin xyz="0.005 0.005 0.013" rpy="0 0 0"/>
-      <geometry>
-        <cylinder length="0.02" radius="0.001"/>
+    <visual>
+      <origin xyz="-0.06 0 0.0" rpy="0 0 0"/>
+      <geometry>
+        <cylinder length="0.5" radius="0.01"/>
+      </geometry>
+      <material name="dark"/>
+    </visual>
+    <collision>
+      <origin xyz="-0.06 0 0.0" rpy="0 0 0"/>
+      <geometry>
+        <cylinder length="0.5" radius="0.01"/>
       </geometry>
     </collision>
   </link>
   <joint name="new_camera_joint" type="fixed">
-    <origin xyz="0.073 -0.011 0.084" rpy="0 0 0"/>
+    <origin xyz="0 0 0.25" rpy="0 0 0"/>
     <parent link="base_link"/>
     <child link="new_camera_link"/>
+  </joint>
+   <link name="new_camera_base_link">
+    <visual>
+      <origin xyz="-0.06 0 0.5" rpy="0 0 0"/>
+      <geometry>
+        <cylinder length="0.01" radius="0.03"/>
+      </geometry>
+      <material name="blue"/>
+    </visual>
+    <collision>
+      <origin xyz="0 0 0.0" rpy="0 0 0"/>
+      <geometry>
+        <cylinder length="0.01" radius="0.03"/>
+      </geometry>
+    </collision>
+  </link>
+  <joint name="new_camera_base_joint" type="fixed">
+    <origin xyz="0 0 0" rpy="0 0 0"/>
+    <parent link="new_camera_link"/>
+    <child link="new_camera_base_link"/>
   </joint>
   <joint name="camera_rgb_joint" type="fixed">

Commit message: a

File: robutler_description_23-24/urdf/robutler.urdf.xacro (robot description, xacro)
@@ -189,5 +189,5 @@
   </link>
   <joint name="new_camera_joint" type="fixed">
-    <origin xyz="0 0 0.25" rpy="0 0 0"/>
+    <origin xyz="-0.06 0 0.34" rpy="0 0 0"/>
     <parent link="base_link"/>
     <child link="new_camera_link"/>
@@ -195,5 +195,5 @@
    <link name="new_camera_base_link">
     <visual>
-      <origin xyz="-0.06 0 0.5" rpy="0 0 0"/>
+      <origin xyz="-0.06 0 0.25" rpy="0 0 0"/>
       <geometry>
         <cylinder length="0.01" radius="0.03"/>
@@ -209,5 +209,5 @@
   </link>
   <joint name="new_camera_base_joint" type="fixed">
-    <origin xyz="0 0 0" rpy="0 0 0"/>
+    <origin xyz="0 0 0.005" rpy="0 0 0"/>
     <parent link="new_camera_link"/>
     <child link="new_camera_base_link"/>

Commit message: new position spwan

File: robutler_description_23-24/urdf/robutler.urdf.xacro (robot description, xacro)
@@ -3,5 +3,5 @@
   <xacro:include filename="$(find robutler_description_23-24)/urdf/common_properties.xacro"/>
   <xacro:include filename="$(find robutler_description_23-24)/urdf/robutler.gazebo.xacro"/>
-  <link name="base_footprint"/>
+  <link name="base_footprint" />
   <joint name="base_joint" type="fixed">
     <parent link="base_footprint"/>
