Commit message: UPDATE Spawn, Photo, Move working with manipulator

File: robutler_description_23_24/urdf/manipulation_robot.urdf.xacro (robot description, xacro)
@@ -4,5 +4,5 @@
   <xacro:include filename="$(find turtlebot3_description)/urdf/turtlebot3_waffle_pi_for_open_manipulator.urdf.xacro"/>
   <!-- Include OpenMANIPULATOR URDF -->
-  <xacro:include filename="$(find turtlebot3_manipulation_description)/urdf/open_manipulator_x.urdf.xacro"/>
+  <xacro:include filename="$(find robutler_description_23_24)/urdf/open_manipulator_x.urdf.xacro"/>
   <!-- Base fixed joint -->
   <joint name="base_fixed" type="fixed">

File: robutler_description_23_24/urdf/open_manipulator_x.urdf.xacro (robot description, xacro)
@@ -2,7 +2,7 @@
 <robot xmlns:xacro="http://ros.org/wiki/xacro">
   <!-- Include OpenManipulator Gazebo Parameter -->
-  <xacro:include filename="$(find turtlebot3_manipulation_description)/urdf/open_manipulator_x.gazebo.xacro"/>
+  <xacro:include filename="$(find robutler_description_23_24)/urdf/open_manipulator_x.gazebo.xacro"/>
   <!-- Include OpenManipulator Transmission -->
-  <xacro:include filename="$(find turtlebot3_manipulation_description)/urdf/open_manipulator_x.transmission.xacro"/>
+  <xacro:include filename="$(find robutler_description_23_24)/urdf/open_manipulator_x.transmission.xacro"/>
   <!-- Link 1 -->
   <link name="link1">
@@ -10,12 +10,12 @@
       <origin xyz="0 0 0" rpy="0 0 0"/>
       <geometry>
-        <mesh filename="package://turtlebot3_manipulation_description/meshes/chain_link1.stl" scale="0.001 0.001 0.001"/>
-      </geometry>
-      <material name="grey"/>
-    </visual>
-    <collision>
-      <origin xyz="0 0 0" rpy="0 0 0"/>
-      <geometry>
-        <mesh filename="package://turtlebot3_manipulation_description/meshes/chain_link1.stl" scale="0.001 0.001 0.001"/>
+        <mesh filename="package://robutler_description_23_24/meshes/chain_link1.stl" scale="0.001 0.001 0.001"/>
+      </geometry>
+      <material name="grey"/>
+    </visual>
+    <collision>
+      <origin xyz="0 0 0" rpy="0 0 0"/>
+      <geometry>
+        <mesh filename="package://robutler_description_23_24/meshes/chain_link1.stl" scale="0.001 0.001 0.001"/>
       </geometry>
     </collision>
@@ -41,5 +41,5 @@
       <origin xyz="0 0 0.018" rpy="0 0 0"/>
       <geometry>
-        <mesh filename="package://turtlebot3_manipulation_description/meshes/chain_link2.stl" scale="0.001 0.001 0.001"/>
+        <mesh filename="package://robutler_description_23_24/meshes/chain_link2.stl" scale="0.001 0.001 0.001"/>
       </geometry>
       <material name="grey"/>
@@ -48,5 +48,5 @@
       <origin xyz="0 0 0.018" rpy="0 0 0"/>
       <geometry>
-        <mesh filename="package://turtlebot3_manipulation_description/meshes/chain_link2.stl" scale="0.001 0.001 0.001"/>
+        <mesh filename="package://robutler_description_23_24/meshes/chain_link2.stl" scale="0.001 0.001 0.001"/>
       </geometry>
     </collision>
@@ -72,12 +72,12 @@
       <origin xyz="0 0 0" rpy="0 0 0"/>
       <geometry>
-        <mesh filename="package://turtlebot3_manipulation_description/meshes/chain_link3.stl" scale="0.001 0.001 0.001"/>
-      </geometry>
-      <material name="grey"/>
-    </visual>
-    <collision>
-      <origin xyz="0 0 0" rpy="0 0 0"/>
-      <geometry>
-        <mesh filename="package://turtlebot3_manipulation_description/meshes/chain_link3.stl" scale="0.001 0.001 0.001"/>
+        <mesh filename="package://robutler_description_23_24/meshes/chain_link3.stl" scale="0.001 0.001 0.001"/>
+      </geometry>
+      <material name="grey"/>
+    </visual>
+    <collision>
+      <origin xyz="0 0 0" rpy="0 0 0"/>
+      <geometry>
+        <mesh filename="package://robutler_description_23_24/meshes/chain_link3.stl" scale="0.001 0.001 0.001"/>
       </geometry>
     </collision>
@@ -103,12 +103,12 @@
       <origin xyz="0 0 0" rpy="0 0 0"/>
       <geometry>
-        <mesh filename="package://turtlebot3_manipulation_description/meshes/chain_link4.stl" scale="0.001 0.001 0.001"/>
-      </geometry>
-      <material name="grey"/>
-    </visual>
-    <collision>
-      <origin xyz="0 0 0" rpy="0 0 0"/>
-      <geometry>
-        <mesh filename="package://turtlebot3_manipulation_description/meshes/chain_link4.stl" scale="0.001 0.001 0.001"/>
+        <mesh filename="package://robutler_description_23_24/meshes/chain_link4.stl" scale="0.001 0.001 0.001"/>
+      </geometry>
+      <material name="grey"/>
+    </visual>
+    <collision>
+      <origin xyz="0 0 0" rpy="0 0 0"/>
+      <geometry>
+        <mesh filename="package://robutler_description_23_24/meshes/chain_link4.stl" scale="0.001 0.001 0.001"/>
       </geometry>
     </collision>
@@ -134,12 +134,12 @@
       <origin xyz="0 0 0" rpy="0 0 0"/>
       <geometry>
-        <mesh filename="package://turtlebot3_manipulation_description/meshes/chain_link5.stl" scale="0.001 0.001 0.001"/>
-      </geometry>
-      <material name="grey"/>
-    </visual>
-    <collision>
-      <origin xyz="0 0 0" rpy="0 0 0"/>
-      <geometry>
-        <mesh filename="package://turtlebot3_manipulation_description/meshes/chain_link5.stl" scale="0.001 0.001 0.001"/>
+        <mesh filename="package://robutler_description_23_24/meshes/chain_link5.stl" scale="0.001 0.001 0.001"/>
+      </geometry>
+      <material name="grey"/>
+    </visual>
+    <collision>
+      <origin xyz="0 0 0" rpy="0 0 0"/>
+      <geometry>
+        <mesh filename="package://robutler_description_23_24/meshes/chain_link5.stl" scale="0.001 0.001 0.001"/>
       </geometry>
     </collision>
@@ -161,5 +161,5 @@
       <origin xyz="0.0 0.0 0" rpy="0 0 0"/>
       <geometry>
-        <mesh filename="package://turtlebot3_manipulation_description/meshes/chain_link_grip_l.stl" scale="0.001 0.001 0.001"/>
+        <mesh filename="package://robutler_description_23_24/meshes/chain_link_grip_l.stl" scale="0.001 0.001 0.001"/>
       </geometry>
       <material name="grey"/>
@@ -168,5 +168,5 @@
       <origin xyz="0.0 0.0 0" rpy="0 0 0"/>
       <geometry>
-        <mesh filename="package://turtlebot3_manipulation_description/meshes/chain_link_grip_l.stl" scale="0.001 0.001 0.001"/>
+        <mesh filename="package://robutler_description_23_24/meshes/chain_link_grip_l.stl" scale="0.001 0.001 0.001"/>
       </geometry>
     </collision>
@@ -192,5 +192,5 @@
       <origin xyz="0.0 -0.0 0" rpy="0 0 0"/>
       <geometry>
-        <mesh filename="package://turtlebot3_manipulation_description/meshes/chain_link_grip_r.stl" scale="0.001 0.001 0.001"/>
+        <mesh filename="package://robutler_description_23_24/meshes/chain_link_grip_r.stl" scale="0.001 0.001 0.001"/>
       </geometry>
       <material name="grey"/>
@@ -199,5 +199,5 @@
       <origin xyz="0.0 -0.0 0" rpy="0 0 0"/>
       <geometry>
-        <mesh filename="package://turtlebot3_manipulation_description/meshes/chain_link_grip_r.stl" scale="0.001 0.001 0.001"/>
+        <mesh filename="package://robutler_description_23_24/meshes/chain_link_grip_r.stl" scale="0.001 0.001 0.001"/>
       </geometry>
     </collision>

Commit message: Updated xacros: color and camera turned 3.14

File: robutler_description_23_24/urdf/manipulation_robot.urdf.xacro (robot description, xacro)
@@ -2,5 +2,5 @@
 <robot name="turtlebot3_manipulation" xmlns:xacro="http://ros.org/wiki/xacro">
   <!-- Include TurtleBot3 Waffle URDF -->
-  <xacro:include filename="$(find turtlebot3_description)/urdf/turtlebot3_waffle_pi_for_open_manipulator.urdf.xacro"/>
+  <xacro:include filename="$(find robutler_description_23_24)/urdf/robutler.urdf.xacro"/>
   <!-- Include OpenMANIPULATOR URDF -->
   <xacro:include filename="$(find robutler_description_23_24)/urdf/open_manipulator_x.urdf.xacro"/>
@@ -11,4 +11,5 @@
     <child link="link1"/>
   </joint>
+  <!--
     <link name="new_camera_link">
     <visual>
@@ -62,4 +63,4 @@
     <child link="camera_rgb_optical_frame2"/>
   </joint>
-  <link name="camera_rgb_optical_frame2"/>
+  <link name="camera_rgb_optical_frame2"/> -->
 </robot>

File: robutler_description_23_24/urdf/open_manipulator_x.gazebo.xacro (robot description, xacro)
@@ -10,5 +10,5 @@
       <maxVel>1.0</maxVel>
       <minDepth>0.001</minDepth>
-      <material>Gazebo/Red</material>
+      <material>Gazebo/FlatBlack</material>
     </gazebo>
   </xacro:macro>
@@ -31,4 +31,5 @@
     <material>Gazebo/DarkGrey</material>
   </gazebo>
+  <!--
   <gazebo reference="new_camera_link">
     <material>Gazebo/DarkGrey</material>
@@ -37,4 +38,5 @@
     <material>Gazebo/FlatBlack</material>
   </gazebo>
+  -->
   <!-- ros_control plugin -->
   <gazebo>

File: robutler_description_23_24/urdf/robutler.gazebo.xacro (robot description, xacro)
@@ -5,11 +5,11 @@
   <xacro:arg name="imu_visual"    default="false"/>
   <gazebo reference="base_link">
-    <material>Gazebo/Red</material>
+    <material>Gazebo/Grey</material>
   </gazebo>
    <gazebo reference="new_camera_link">
-    <material>Gazebo/Red</material>
+    <material>Gazebo/Grey</material>
   </gazebo>
    <gazebo reference="new_camera_base_link">
-    <material>Gazebo/FlatBlack</material>
+    <material>Gazebo/Grey</material>
   </gazebo>
   <gazebo reference="wheel_left_link">
@@ -109,5 +109,5 @@
   </gazebo>
   <gazebo reference="base_scan">
-    <material>Gazebo/Blue</material>
+    <material>Gazebo/White</material>
     <sensor type="ray" name="lds_lfcd_sensor">
       <pose>0 0 0 0 0 </pose>
@@ -144,4 +144,5 @@
     <sensor type="camera" name="Pi Camera">
       <always_on>true</always_on>
+      <pose>0 0 0 0 0 3.14</pose>
       <visualize>$(arg camera_visual)</visualize>
       <camera>

File: robutler_description_23_24/urdf/robutler.urdf.xacro (robot description, xacro)
@@ -199,5 +199,5 @@
         <cylinder length="0.01" radius="0.03"/>
       </geometry>
-      <material name="blue"/>
+      <material name="green"/>
     </visual>
     <collision>
@@ -226,6 +226,6 @@
   <link name="camera_rgb_optical_frame2"/>
   <joint name="camera_rgb_joint" type="fixed">
-    <origin xyz="0.003 0.011 0.009" rpy="0 0 0"/>
-    <parent link="camera_link"/>
+    <origin xyz="-0.06 0 0.6" rpy="0 0 3.14"/>
+    <parent link="new_camera_base_link"/>
     <child link="camera_rgb_frame"/>
   </joint>
